File: InverSol_ESP32.sch (KiCad schematic (older format))
At the start: 3 parts, among them J1 Conn_02x20_Odd_Even, U1 ESP32-WROOM

Commit message: added some new lib stuff
Connections:
- net +3V3: now also J1.3 (Pin_3), J1.4 (Pin_4)
- net GND: now also J1.5 (Pin_5), J1.6 (Pin_6), J1.7 (Pin_7)
- net IO25: now reaches U1.10 (IO25)
- net IO25: now also J1.23 (Pin_23)
- net IO26: now reaches U1.11 (IO26)
- net IO26: now also J1.25 (Pin_25)
- net IO27: now reaches U1.12 (IO27)
- net IO27: now also J1.27 (Pin_27)
- net IO14: now reaches U1.13 (IO14)
- net IO14: now also J1.29 (Pin_29)
- net IO12: now reaches U1.14 (IO12)
- net IO12: now also J1.31 (Pin_31)
- net IO13: now reaches U1.16 (IO13)
- net IO13: now also J1.40 (Pin_40)
- net SD2/IO9: now reaches U1.17 (SD2/IO9)
- net SD2/IO9: now also J1.35 (Pin_35)
- net SD3/IO10: now reaches U1.18 (SD3/IO10)
- net SD3/IO10: now also J1.33 (Pin_33)
- net CMD/IO11: now reaches U1.19 (CMD/IO11)
- net CMD/IO11: now also J1.38 (Pin_38)
- net CLK/IO6: now reaches U1.20 (CLK/IO6)
- net CLK/IO6: now also J1.36 (Pin_36)
- net SD0/IO7: now reaches U1.21 (SD0/IO7)
- net SD0/IO7: now also J1.39 (Pin_39)
- net SD1/IO8: now reaches U1.22 (SD1/IO8)
- net SD1/IO8: now also J1.37 (Pin_37)
- net IO15: now reaches U1.23 (IO15)
- net IO15: now also J1.34 (Pin_34)
- net IO2: now reaches U1.24 (IO2)
- net IO2: now also J1.32 (Pin_32)
- net IO0: now reaches U1.25 (IO0)
- net IO0: now also J1.30 (Pin_30)
- net IO4: now reaches U1.26 (IO4)
- net IO4: now also J1.28 (Pin_28)
- net IO16: now reaches U1.27 (IO16)
- net IO16: now also J1.26 (Pin_26)
- net IO17: now reaches U1.28 (IO17)
- net IO17: now also J1.24 (Pin_24)
- net IO5: now reaches U1.29 (IO5)
- net IO5: now also J1.22 (Pin_22)
- net IO18: now reaches U1.30 (IO18)
- net IO18: now also J1.20 (Pin_20)
- net IO19: now reaches U1.31 (IO19)
- net IO19: now also J1.18 (Pin_18)
- net IO21: now reaches U1.33 (IO21)
- net IO21: now also J1.16 (Pin_16)
- net RXD0: now reaches U1.34 (RXD0)
- net RXD0: now also J1.14 (Pin_14)
- net TXD0: now reaches U1.35 (TXD0)
- net TXD0: now also J1.12 (Pin_12)
- net IO22: now reaches U1.36 (IO22)
- net IO22: now also J1.10 (Pin_10)
- net IO23: now reaches U1.37 (IO23)
- net IO23: now also J1.8 (Pin_8)
- net SENSOR_VP: now reaches U1.4 (SENSOR_VP)
- net SENSOR_VP: now also J1.11 (Pin_11)
- net SENSOR_VN: now reaches U1.5 (SENSOR_VN)
- net SENSOR_VN: now also J1.13 (Pin_13)
- net IO34: now reaches U1.6 (IO34)
- net IO34: now also J1.15 (Pin_15)
- net IO35: now reaches U1.7 (IO35)
- net IO35: now also J1.17 (Pin_17)
- net IO32: now reaches U1.8 (IO32)
- net IO32: now also J1.19 (Pin_19)
- net IO33: now reaches U1.9 (IO33)
- net IO33: now also J1.21 (Pin_21)
- net Vin: now reaches J1.1 (Pin_1)
- net Vin: now also J1.2 (Pin_2)
- net EN: now reaches J1.9 (Pin_9)
Other:
- note added: "ESP32-WROOM-32"
- note added: "Note:\nVin around 24V from InverSol Batteries"

Commit message: added psupply and calc spreadsheet
Parts:
- added C1, C2, C3: C, symbol C
- added D1: D_Zener_ALT, symbol D_Zener_ALT
- added L1: L, symbol L
- added R2, R3: R, symbol R
- added U?: LM2675, symbol LM2675
Connections:
- net +3V3: now also C2.1, L1.2, R3.1
- net GND: now also C2.2, C3.2, D1.2 (A), R2.2, U?.6 (GND)
- new net: C1.1, U?.1 (C_B)
- new net: R2.1, R3.2, U?.4 (FB)
- new net: C1.2, D1.1 (K), L1.1, U?.8 (V_SW)
- new net VBATT: C3.1, U?.7 (V_IN)
Other:
- note added: "GPIO Connector"
- note added: "NOTES:\n-Locate Programming Resistors near the Feedback Pin using Short Leads\n-Heavy Lines Must Be Kept Short and Use Ground Plane Construction for Best Results"
- note added: "Power Supply"
Changed lines of the file:
@@
 $EndComp
 Text Notes 1650 9200 0    157  ~ 31
-Espressif ESP-WROOM-32 MODULE
+GPIO Connector
 $Comp
 L Conn_02x20_Odd_Even J1
@@
 	0    -1   -1   0
 $EndComp
+Text Notes 8050 3800 0    60   ~ 0
+ESP32-WROOM-32
+$Comp
+L LM2675 U?
+U 1 1 5B1ADF0F
+P 15600 5100
+F 0 "U?" H 15600 5100 60  0000 C CNN
+F 1 "LM2675" H 15550 5300 60  0000 C CNN
+F 2 "" H 15600 5100 60  0000 C CNN
+F 3 "" H 15600 5100 60  0000 C CNN
+	1    15600 5100
+	1    0    0    -1
+$EndComp
+$Comp
+L R R3
+U 1 1 5B1AE6F0
+P 16150 4300
+F 0 "R3" V 16230 4300 50  0000 C CNN
+F 1 "R" V 16150 4300 50  0000 C CNN
+F 2 "" V 16080 4300 50  0001 C CNN
+F 3 "" H 16150 4300 50  0001 C CNN
+	1    16150 4300
+	0    1    1    0
+$EndComp
+$Comp
+L R R2
+U 1 1 5B1AE9F3
+P 15650 4300
+F 0 "R2" V 15730 4300 50  0000 C CNN
+F 1 "R" V 15650 4300 50  0000 C CNN
+F 2 "" V 15580 4300 50  0001 C CNN
+F 3 "" H 15650 4300 50  0001 C CNN
+	1    15650 4300
+	0    1    1    0
+$EndComp
+$Comp
+L C C3
+U 1 1 5B1AEA34
+P 14450 5500
+F 0 "C3" H 14475 5600 50  0000 L CNN
+F 1 "C" H 14475 5400 50  0000 L CNN
+F 2 "" H 14488 5350 50  0001 C CNN
+F 3 "" H 14450 5500 50  0001 C CNN
+	1    14450 5500
+	1    0    0    -1
+$EndComp
+$Comp
+L C C2
+U 1 1 5B1AEA85
+P 17450 5500
+F 0 "C2" H 17475 5600 50  0000 L CNN
+F 1 "C" H 17475 5400 50  0000 L CNN
+F 2 "" H 17488 5350 50  0001 C CNN
+F 3 "" H 17450 5500 50  0001 C CNN
+	1    17450 5500
+	1    0    0    -1
+$EndComp
+$Comp
+L C C1
+U 1 1 5B1AEAE6
+P 16800 4900
+F 0 "C1" H 16825 5000 50  0000 L CNN
+F 1 "C" H 16825 4800 50  0000 L CNN
+F 2 "" H 16838 4750 50  0001 C CNN
+F 3 "" H 16800 4900 50  0001 C CNN
+	1    16800 4900
+	1    0    0    -1
+$EndComp
+$Comp
+L D_Zener_ALT D1
+U 1 1 5B1AEB21
+P 16800 5450
+F 0 "D1" H 16800 5550 50  0000 C CNN
+F 1 "D_Zener_ALT" H 16800 5350 50  0000 C CNN
+F 2 "" H 16800 5450 50  0001 C CNN
+F 3 "" H 16800 5450 50  0001 C CNN
+	1    16800 5450
+	0    1    1    0
+$EndComp
 Wire Notes Line
 	1550 1400 11600 1400
@@
 Wire Wire Line
 	6700 11400 6750 11400
-Text Notes 8050 3800 0    60   ~ 0
-ESP32-WROOM-32
+Wire Wire Line
+	15900 4400 15900 4300
+Wire Wire Line
+	15800 4300 16000 4300
+Connection ~ 15900 4300
+Wire Wire Line
+	16600 5000 16600 4750
+Wire Wire Line
+	16600 4750 16800 4750
+Wire Wire Line
+	16600 5200 16950 5200
+Wire Wire Line
+	16800 5050 16800 5300
+$Comp
+L L L1
+U 1 1 5B1AF1BD
+P 17100 5200
+F 0 "L1" V 17050 5200 50  0000 C CNN
+F 1 "L" V 17175 5200 50  0000 C CNN
+F 2 "" H 17100 5200 50  0001 C CNN
+F 3 "" H 17100 5200 50  0001 C CNN
+	1    17100 5200
+	0    -1   -1   0
+$EndComp
+Connection ~ 16800 5200
+Wire Wire Line
+	17450 4150 17450 5350
+Wire Wire Line
+	17450 5200 17250 5200
+Wire Wire Line
+	17450 4300 16300 4300
+Connection ~ 17450 5200
+$Comp
+L +3V3 #PWR?
+U 1 1 5B1AF69C
+P 17450 4150
+F 0 "#PWR?" H 17450 4000 50  0001 C CNN
+F 1 "+3V3" H 17450 4290 50  0000 C CNN
+F 2 "" H 17450 4150 50  0001 C CNN
+F 3 "" H 17450 4150 50  0001 C CNN
+	1    17450 4150
+	1    0    0    -1
+$EndComp
+Connection ~ 17450 4300
+Wire Wire Line
+	15300 5800 15300 6100
+Wire Wire Line
+	14450 5650 14450 6250
+Connection ~ 15900 6250
+Wire Wire Line
+	15900 5800 15900 6350
+Wire Wire Line
+	16800 6250 16800 5600
+Wire Wire Line
+	17450 6250 17450 5650
+Connection ~ 16800 6250
+Wire Wire Line
+	14450 5350 14450 5100
+Wire Wire Line
+	14050 5100 14600 5100
+Connection ~ 14450 5100
+Text Label 14050 5100 0    60   ~ 0
+VBATT
+Connection ~ 14450 6250
+Wire Wire Line
+	14450 6250 17450 6250
+$Comp
+L GND #PWR?
+U 1 1 5B1B017D
+P 15900 6350
+F 0 "#PWR?" H 15900 6100 50  0001 C CNN
+F 1 "GND" H 15900 6200 50  0000 C CNN
+F 2 "" H 15900 6350 50  0001 C CNN
+F 3 "" H 15900 6350 50  0001 C CNN
+	1    15900 6350
+	1    0    0    -1
+$EndComp
+$Comp
+L GND #PWR?
+U 1 1 5B1B01A7
+P 15350 4300
+F 0 "#PWR?" H 15350 4050 50  0001 C CNN
+F 1 "GND" H 15350 4150 50  0000 C CNN
+F 2 "" H 15350 4300 50  0001 C CNN
+F 3 "" H 15350 4300 50  0001 C CNN
+	1    15350 4300
+	0    1    1    0
+$EndComp
+Wire Wire Line
+	15350 4300 15500 4300
+Wire Notes Line
+	12600 1400 12600 8400
+Wire Notes Line
+	12600 8400 19650 8400
+Wire Notes Line
+	19650 8400 19650 1400
+Wire Notes Line
+	19650 1400 12600 1400
+Text Notes 12700 1700 0    157  ~ 31
+Power Supply
+Text Notes 12700 8250 0    60   ~ 0
+NOTES:\n-Locate Programming Resistors near the Feedback Pin using Short Leads\n-Heavy Lines Must Be Kept Short and Use Ground Plane Construction for Best Results
 $EndSCHEMATC
